Commit message: working model on 29/June/2023

File: src/robot_arm_urdf/urdf/robot_arm_urdf.urdf (robot description, URDF)
Before this commit: robot robot_arm_urdf, 15 links, 14 joints
Links:
- link gripper_finger1_finger_tip_link: mass 0.0124305 -> 0.010005
- link gripper_finger2_finger_tip_link: mass 0.0124305 -> 0.010005

Commit message: Added updated src fle

File: src/robot_arm_urdf/urdf/robot_arm_urdf.urdf (robot description, URDF)
Before this commit: robot robot_arm_urdf, 15 links, 14 joints
Joints:
- joint joint_1: limit lower=0 upper=3.142 effort=300 velocity=3 -> lower=-3.14 upper=3.142 effort=300 velocity=3
